File: accelerometer.kicad_sch (KiCad schematic)
At the start: 5 parts, among them U4 BMA400

Commit message: Add new mcu and better leds layout
Parts:
- renumbered C17 to C21, C18 to C22
Changed lines of the file:
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@@
 	(generator_version "9.0")
 	(paper "A5")
+	(title_block
+		(date "2025-12-21")
+	)
 	(junction
 		(at 168.91 41.91)
@@
 		(on_board yes)
 		(dnp no)
-		(property "Reference" "C18"
+		(property "Reference" "C22"
 			(at 166.37 54.864 90)
 			(effects
@@
 			(project "Eval_boards"
 				(path "/d7ecb1f3-4916-4ecb-8c6e-b89f175440e1/8b5c4eb3-9c02-477c-8af4-4b02c637b128"
-					(reference "C18")
+					(reference "C22")
 					(unit 1)
 				)
@@
 		(on_board yes)
 		(dnp no)
-		(property "Reference" "C17"
+		(property "Reference" "C21"
 			(at 158.75 54.864 90)
 			(effects
@@
 			(project "Eval_boards"
 				(path "/d7ecb1f3-4916-4ecb-8c6e-b89f175440e1/8b5c4eb3-9c02-477c-8af4-4b02c637b128"
-					(reference "C17")
+					(reference "C21")
 					(unit 1)
 				)
